Commit message: add bumper for turtlebot3

File: urdf/turtlebot3_waffle.gazebo.xacro (robot description, xacro)
@@ -177,3 +177,23 @@
     </sensor>
   </gazebo>
+  <gazebo reference="bumper_link">
+    <sensor name="contacts" type="contact">
+        <contact>
+          <collision>base_footprint_fixed_joint_lump__base_collision_collision_1</collision>
+        </contact>
+        <plugin name="gazebo_ros_bumper_controller" filename="libgazebo_ros_bumper.so">
+          <always_on>true</always_on>
+          <robotNamespace>/robot</robotNamespace>
+          <bumperTopicName>bumper_states</bumperTopicName>
+          <frameName>bumper</frameName>
+          <visualize>true</visualize>
+          <update_rate>50.0</update_rate>
+        </plugin>
+    </sensor>
+    <material>Gazebo/Red</material>
+    <mu1>0.1</mu1>
+    <mu2>0.1</mu2>
+    <gravity>true</gravity>
+    <selfCollide>false</selfCollide>
+  </gazebo>
 </robot>

File: urdf/turtlebot3_waffle.urdf.xacro (robot description, xacro)
@@ -35,4 +35,31 @@
     </inertial>
   </link>
+  <link name="bumper_link">
+    <inertial>
+        <origin xyz="0.0 0.0 0.0" rpy="0 1.0 0"/>
+        <mass value="0.0000000001"/>
+        <inertia ixx="0.00000001" ixy="0.00000001" ixz="0.00000001" iyy="0.00000001" iyz="0.00000001" izz="0.00000001"/>
+    </inertial>
+    <visual>
+        <origin xyz="0.0 0.0 0.0" rpy="0.0 1.0 0"/>
+        <geometry>
+            <cylinder radius="0.01" length="0.01"/>
+        </geometry>
+        <material name="red">
+            <color rgba="1.0 0.0 0.0 1.0"/>
+        </material>
+    </visual>
+    <collision name="base_collision">
+        <origin xyz="0.0 0.0 0.0" rpy="0.0 1.0 0.0"/>
+        <geometry>
+            <cylinder radius="0.01" length="0.01"/>
+        </geometry>
+    </collision>
+  </link>
+  <joint name="bumper_joint" type="fixed">
+      <origin xyz="0.075 0.0 0.1" rpy="0.0 0.0 0.0"/>
+      <parent link="base_link"/>
+      <child link="bumper_link"/>
+  </joint>
   <joint name="wheel_left_joint" type="continuous">
     <parent link="base_link"/>
